Commit message: 删去waffle模型的无用信息

File: src/my_navigation_simulation/mybot_description/urdf/mybot_waffle.gazebo.xacro (robot description, xacro)
@@ -3,5 +3,4 @@
     xmlns:xacro="http://ros.org/wiki/xacro">
     <xacro:arg name="gpu" default="true"/>
-    <!-- <xacro:arg name="laser_visual" default="false"/> -->
     <xacro:arg name="camera_visual" default="false"/>
     <xacro:arg name="imu_visual" default="false"/>
@@ -20,5 +19,25 @@
         <material>Gazebo/FlatBlack</material>
     </gazebo>
+    <gazebo reference="wheel_leftback_link">
+        <mu1>0.1</mu1>
+        <mu2>0.1</mu2>
+        <kp>500000.0</kp>
+        <kd>10.0</kd>
+        <minDepth>0.001</minDepth>
+        <maxVel>0.1</maxVel>
+        <fdir1>1 0 0</fdir1>
+        <material>Gazebo/FlatBlack</material>
+    </gazebo>
     <gazebo reference="wheel_right_link">
+        <mu1>0.1</mu1>
+        <mu2>0.1</mu2>
+        <kp>500000.0</kp>
+        <kd>10.0</kd>
+        <minDepth>0.001</minDepth>
+        <maxVel>0.1</maxVel>
+        <fdir1>1 0 0</fdir1>
+        <material>Gazebo/FlatBlack</material>
+    </gazebo>
+    <gazebo reference="wheel_rightback_link">
         <mu1>0.1</mu1>
         <mu2>0.1</mu2>
@@ -105,36 +124,4 @@
         </plugin>
     </gazebo>
-    <!-- <gazebo reference="base_scan">
-        <material>Gazebo/FlatBlack</material>
-        <sensor type="ray" name="lds_lfcd_sensor">
-            <pose>0 0 0 0 0 0</pose>
-            <visualize>$(arg laser_visual)</visualize>
-            <update_rate>5</update_rate>
-            <ray>
-                <scan>
-                    <horizontal>
-                        <samples>360</samples>
-                        <resolution>1</resolution>
-                        <min_angle>0.0</min_angle>
-                        <max_angle>6.28319</max_angle>
-                    </horizontal>
-                </scan>
-                <range>
-                    <min>0.120</min>
-                    <max>3.5</max>
-                    <resolution>0.015</resolution>
-                </range>
-                <noise>
-                    <type>gaussian</type>
-                    <mean>0.0</mean>
-                    <stddev>0.01</stddev>
-                </noise>
-            </ray>
-            <plugin name="gazebo_ros_lds_lfcd_controller" filename="libgazebo_ros_laser.so">
-                <topicName>scan</topicName>
-                <frameName>base_scan</frameName>
-            </plugin>
-        </sensor>
-    </gazebo> -->
     <gazebo reference="camera_rgb_frame">
         <sensor type="depth" name="realsense_R200">

File: src/my_navigation_simulation/mybot_description/urdf/mybot_waffle.urdf.xacro (robot description, xacro)
@@ -130,33 +130,8 @@
     </joint>
     <link name="imu_link"/>
-    <!-- <joint name="scan_joint" type="fixed">
-        <parent link="base_link"/>
-        <child link="base_scan"/>
-        <origin xyz="-0.064 0 0.122" rpy="0 0 0"/>
-    </joint> -->
     <xacro:include filename="$(find velodyne_description)/urdf/HDL-32E.urdf.xacro"/>
     <xacro:HDL-32E parent="base_link" name="velodyne" topic="/velodyne_points" hz="10" samples="220" gpu="${gpu}">
         <origin xyz="-0.07 0.0 0.093" rpy="0 0 0" />
     </xacro:HDL-32E>
-    <!-- <link name="base_scan">
-        <visual>
-            <origin xyz="0 0 0" rpy="0 0 0"/>
-            <geometry>
-                <mesh filename="package://turtlebot3_description/meshes/sensors/lds.stl" scale="0.001 0.001 0.001"/>
-            </geometry>
-            <material name="dark"/>
-        </visual>
-        <collision>
-            <origin xyz="0.015 0 -0.0065" rpy="0 0 0"/>
-            <geometry>
-                <cylinder length="0.0315" radius="0.055"/>
-            </geometry>
-        </collision>
-        <inertial>
-            <mass value="0.114" />
-            <origin xyz="0 0 0" />
-            <inertia ixx="0.001" ixy="0.0" ixz="0.0" iyy="0.001" iyz="0.0" izz="0.001" />
-        </inertial>
-    </link> -->
     <joint name="camera_joint" type="fixed">
         <origin xyz="0.064 -0.065 0.094" rpy="0 0 0"/>
